File: starterProject_kiCad/starterProject.kicad_pcb (KiCad board)
At the start: 2 copper layers, 50.7 x 50.7 mm, 16 parts, among them J1 Screw_Terminal_01x02, J2 Programming Connector, SW1 SW_Push, U1 PIC12LF1501

Commit message: added decore silkscreen and gerber
Parts:
- added G***: LOGO, Tutorial_Footprints:Logo_SilkScreen_15mm, F.Cu at (109.7, 79.8)
- added G***: LOGO, Tutorial_Footprints:Logo_Horizontal_Silkscreen_10mm, B.Cu at (119.9, 75.2)
- moved SW1 1.47 mm to (111.5, 93.2)
Routing:
- net Net-(SW1-Pad2): track 25.3 -> 23.2 mm
Other:
- board text added: "2023 Electrical Tutorial Huan Yi Shen 2023-02-14"
- board text added: "3V3"
- board text added: "3V3 ~{MCLR}"
- board text added: "GND"
- board text added: "TOP"
